Commit message: updated config loading logic and urdf offset

File: alicia_duo_leader_dashboard/static/robot/model.urdf (robot description, URDF)
Before this commit: robot Alicia_D_v5_6_leader_ur, 8 links, 7 joints
Joints:
- joint joint3: origin xyz=0.18922 0.027473 -0.00041 rpy=0 3.14159 0.7854 -> xyz=0.18922 0.027473 -0.00041 rpy=0 3.14159 0.6109
